File: Hardware/Vorlage ATmega2560-16AU/Vorlage ATmega2560-16AU.brd (EAGLE design)
At the start: 160 x 100 mm, 152 parts, among them IC1 CD74HC14PW, IC2 ATMEGA2560640V-8AU, IC3 SS39E, IC4 SS39E, IC5 74AC138D, IC6 XC6210B332MR, Q1 16MHz, Q10 PMV27UPER, Q2 32.768kHz, Q3 PMV27UPER, Q4 PMV27UPER, Q5 PMV27UPER, Q6 PMV27UPER, Q7 PMV27UPER, Q8 PMV27UPER, Q9 PMV27UPER, U1 LM35DZ, X1 2510-, X2 +5V, X3 2514-, X4 2510-, X5 2510-

Commit message: Bauteile auf 0805
Parts:
- removed R10: 10k, rcl:R1206
- added R37: 10k, rcl:R0805
- C1, C10, C11, C12, C13, C19, C2, C20, C21, C22, C23, C3, C4, C5, C7: device rcl:C1206 -> rcl:C0805
- R11, R12, R14, R15, R16, R18, R19, R2, R20, R21, R22, R23, R24, R25, R26, R28, R29, R3, R30, R31, R32, R33, R34, R35, R36, R4, R45, R5, R7, R8, R9: device rcl:R1206 -> rcl:R0805
- moved R7 919.5 mm to (-130.0, -790.0)
- moved R5 909.6 mm to (-130.0, -780.0)
- moved R2 899.7 mm to (-130.0, -770.0)
- moved R36 898.1 mm to (-130.0, -760.0)
- moved R35 888.6 mm to (-130.0, -750.0)
- moved R34 879.1 mm to (-130.0, -740.0)
- moved R33 869.7 mm to (-130.0, -730.0)
- moved R32 860.4 mm to (-130.0, -720.0)
- moved R31 851.1 mm to (-130.0, -710.0)
- moved R30 841.9 mm to (-130.0, -700.0)
- moved R29 832.8 mm to (-130.0, -690.0)
- moved C12 662.2 mm to (-130.0, -530.0)
- moved C7 654.7 mm to (-130.0, -520.0)
- moved C5 646.9 mm to (-130.0, -510.0)
- moved C4 638.2 mm to (-130.0, -500.0)
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Connections:
- net ADC12: now also R26.2; no longer R26.1
- net N$19: now also R26.1; no longer R26.2
- net N$23: now also R9.2; no longer R9.1
- net N$24: now also R8.2; no longer R8.1
- net N$60: now also R11.2; no longer R11.1
- net N$9: now also R45.2; no longer R45.1
- net RESET: now also R37.1; no longer R10.1
- net VCC: now also R11.1, R37.2, R45.1, R8.1, R9.1; no longer R10.2, R11.2, R45.2, R8.2, R9.2
