File: Hardware/Vorlage ATmega2560-16AU/Vorlage ATmega2560-16AU.sch (EAGLE design)
At the start: 152 parts, among them IC1 CD74HC14PW, IC2 ATMEGA2560640V-8AU, IC3 SS39E, IC4 SS39E, IC5 74AC138D, IC6 XC6210B332MR, Q1 16MHz, Q10 PMV27UPER, Q2 32.768kHz, Q3 PMV27UPER, Q4 PMV27UPER, Q5 PMV27UPER, Q6 PMV27UPER, Q7 PMV27UPER, Q8 PMV27UPER, Q9 PMV27UPER, U1 LM35DZ, X1 2510-, X2 +5V, X3 2514-, X4 2510-, X5 2510-

Commit message: Bauteile auf 0805
Parts:
- removed R10: 10k, rcl:R-EU_R1206
- added R37: 10k, rcl:R-EU_R0805
- C1, C10, C11, C12, C13, C19, C2, C20, C21, C22, C23, C3, C4, C5, C7: device rcl:C-EUC1206 -> rcl:C-EUC0805
- R11, R12, R14, R15, R16, R18, R19, R2, R20, R21, R22, R23, R24, R25, R26, R28, R29, R3, R30, R31, R32, R33, R34, R35, R36, R4, R45, R5, R7, R8, R9: device rcl:R-EU_R1206 -> rcl:R-EU_R0805
Connections:
- net ADC12: now also R26.2; no longer R26.1
- net N$19: now also R26.1; no longer R26.2
- net N$23: now also R9.2; no longer R9.1
- net N$24: now also R8.2; no longer R8.1
- net N$60: now also R11.2; no longer R11.1
- net N$9: now also R45.2; no longer R45.1
- net RESET: now also R37.1; no longer R10.1
- net VCC: now also R11.1, R37.2, R45.1, R8.1, R9.1; no longer R10.2, R11.2, R45.2, R8.2, R9.2
Other:
- moved on the sheet: R11, R26, R45, R8, R9
